File: hardware/PUTM_EV_STEERING_WHEEL_2026/driver_input.kicad_sch (KiCad schematic)
At the start: 36 parts, among them SW1 RTD, SW2 TSA, SW3 CS, SW4 DRS, SW5 ENTER, SW6 BACK, SW7 UP, SW8 DOWN, SW9 RADIO

Commit message: Edit MCU G0->G4, add RS in schema
Parts:
- removed C12: 1u, Capacitor_SMD:C_0603_1608Metric, symbol Device:C_Small
- removed R21: 1k, Resistor_SMD:R_0603_1608Metric, symbol Device:R_Small
- removed R29: 10k, Resistor_SMD:R_0603_1608Metric, symbol Device:R_Small
- added C20, C21, C22, C23, C34, C35, C38, C39, C41, C42, C43, C44, C45, C46, C47, C48: 1u, Capacitor_SMD:C_0603_1608Metric, symbol Device:C_Small
- added J4: M80-5102042, Samacsys:M80-51020YY, symbol Harwin:M80-5102042
- added J5: M80-51014XX, Samacsys:M80-51014YY, symbol Harwin:M80-51014XX
- added R33, R34, R35, R36, R37, R38, R39, R40, R51, R52, R53, R54, R55, R56, R57, R58: 10k, Resistor_SMD:R_0603_1608Metric, symbol Device:R_Small
- added R41, R42, R43, R44, R45, R46, R47, R48, R59, R60, R61, R62, R63, R64, R65, R66: 1k, Resistor_SMD:R_0603_1608Metric, symbol Device:R_Small
Connections:
- net BACK_BTN: now also J5.5 (Pin_5)
- net DOWN_BTN: now also J5.7 (Pin_7)
- net DRS_BTN: now also J5.3 (Pin_3)
- net ENTER_BTN: now also J5.4 (Pin_4)
- net GND: now also C20.2, C21.2, C22.2, C23.2, C34.2, C35.2, C38.2, C39.2, C41.2, C42.2, C43.2, C44.2, C45.2, C46.2, C47.2, C48.2, J4.10, J4.20, J5.9 (Pin_9)
- net RADIO_BTN: now also J5.8 (Pin_8)
- net RTD_BTN: now also J5.1 (Pin_1)
- net TSA_BTN: now also J5.2 (Pin_2)
- net UP_BTN: now also J5.6 (Pin_6)
- new net +5V: R33.1, R34.1, R35.1, R36.1, R37.1, R38.1, R39.1, R40.1, R51.1, R52.1, R53.1, R54.1, R55.1, R56.1, R57.1, R58.1
- new net RS1_1: C39.1, J4.1, R40.2, R41.1, R41.2
- new net RS1_2: C38.1, J4.2, R39.2, R42.1, R42.2
- new net RS1_3: C35.1, J4.3, R38.2, R43.1, R43.2
- new net RS1_4: C34.1, J4.4, R37.2, R44.1, R44.2
- new net RS1_5: C23.1, J4.5, R36.2, R45.1, R45.2
- new net RS1_6: C22.1, J4.6, R35.2, R46.1, R46.2
- new net RS1_7: C21.1, J4.7, R34.2, R47.1, R47.2
- new net RS1_8: C20.1, J4.8, R33.2, R48.1, R48.2
- new net RS2_1: C48.1, J4.11, R58.2, R59.1, R59.2
- new net RS2_2: C47.1, J4.12, R57.2, R60.1, R60.2
- new net RS2_3: C46.1, J4.13, R56.2, R61.1, R61.2
- new net RS2_4: C45.1, J4.14, R55.2, R62.1, R62.2
- new net RS2_5: C44.1, J4.15, R54.2, R63.1, R63.2
- new net RS2_6: C43.1, J4.16, R53.2, R64.1, R64.2
- new net RS2_7: C42.1, J4.17, R52.2, R65.1, R65.2
- new net RS2_8: C41.1, J4.18, R51.2, R66.1, R66.2
Other:
- note added: "BUTTONS"
- note added: "Rotary Switch"
- note added: "To trash"
- note removed: "TODO:"
- note removed: "Znaleźć pokrętła"
- moved on the sheet: C10, C11, C13, C17, C6, C7, C8, C9, R10, R18, R19, R20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
